File: hardware/usb/at90usb162/at90usb162.kicad_pcb (KiCad board)
At the start: 2 copper layers, 47.5 x 44.9 mm, 23 parts, among them IC1 AT90USB162-A, J1 USERPORT, P1 USB, P2 RESET, X1 8Mhz

Commit message: Hardware: Added jumper to configure/adapt C64/C128 reset lines
On the C64 this jumper simply needs to be closed to allow resets. No copper
on the front layer around the pins to allow easy bridging.

On the C128, the reset signal at the userport only resets peripherals. The
jumper needs to be left open, and a wire must be run from the top pin to the
real reset line of the C128 to support hardware resets.
Parts:
- added JP1: JUMPER, PIN_ARRAY_2X1, F.Cu at (198.6, 133.7)
- moved P2 6.38 mm to (191.4, 135.0)
Connections:
- J1 pad 3: /RESET -> /EXTRES
Routing:
- net /EXTRES: track 0.00 -> 38.4 mm, vias 0 -> 1
- net /RESET: track 32.9 -> 8.40 mm, vias 1 -> 0
- net /ATRESET: track 5.73 -> 17.8 mm
- net /D7: track 26.4 -> 30.7 mm

Commit message: Hardware: Changed to rev3, improved component layout
Increased the distance between R1 and R2 because they didn't fit nicely
when using resistors with slightly larger bodies.
Parts:
- moved R3 3.20 mm to (218.6, 128.2), turned to 270 degrees
- moved C3 2.67 mm to (204.1, 128.2)
- moved C5 1.31 mm to (215.3, 128.2), turned to 270 degrees
- moved R1 0.51 mm to (208.8, 128.2)
- moved R2 0.50 mm to (211.8, 128.2)
Routing:
- net GND: track 20.3 -> 25.4 mm
- net N-000008: track 3.29 -> 5.76 mm
Changed lines of the file:
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@@
 (kicad_pcb (version 3) (host pcbnew "(2013-07-07 BZR 4022)-stable")
   (general
-    (links 54)
+    (links 0)
     (no_connects 0)
     (area 169.165002 108.332599 244.854401 163.8376)
     (thickness 1.6)
-    (drawings 50)
-    (tracks 143)
+    (drawings 54)
+    (tracks 148)
     (zones 0)
     (modules 24)
@@
   (title_block
     (title "xlink usb adapter")
-    (rev 2)
+    (rev 3)
     (company "Henning Bekel")
   )
@@
   )
   (module C1 (layer F.Cu)
-    (at 206.7687 128.2319 90)
+    (at 204.1017 128.2319 90)
     (descr "Condensateur e = 1 pas")
     (tags C)
@@
   )
   (module C1 (layer F.Cu)
-    (at 215.6587 126.9619)
+    (at 215.3412 128.2319 270)
     (descr "Condensateur e = 1 pas")
     (tags C)
-    (fp_text reference C5 (at 3.7211 0.0889) (layer F.SilkS)
+    (fp_text reference C5 (at 3.7211 0.0889 270) (layer F.SilkS)
       (effects (font (size 1.016 1.016) (thickness 0.2032)))
     )
-    (fp_text value 4.7nF (at 4.7625 -1.2827) (layer F.SilkS) hide
+    (fp_text value 4.7nF (at 4.7625 -1.2827 270) (layer F.SilkS) hide
       (effects (font (size 1.016 1.016) (thickness 0.2032)))
     )
@@
     (fp_line (start -2.54 1.27) (end -2.54 -1.27) (layer F.SilkS) (width 0.3048))
     (fp_line (start -2.54 -0.635) (end -1.905 -1.27) (layer F.SilkS) (width 0.3048))
-    (pad 1 thru_hole circle (at -1.27 0) (size 1.397 1.397) (drill 0.8128)
+    (pad 1 thru_hole circle (at -1.27 0 270) (size 1.397 1.397) (drill 0.8128)
       (layers *.Cu *.Mask F.SilkS)
       (net 25 /SHIELD)
     )
-    (pad 2 thru_hole circle (at 1.27 0) (size 1.397 1.397) (drill 0.8128)
+    (pad 2 thru_hole circle (at 1.27 0 270) (size 1.397 1.397) (drill 0.8128)
       (layers *.Cu *.Mask F.SilkS)
       (net 27 GND)
@@
   )
   (module R1 (layer F.Cu)
-    (at 209.3214 128.2319 270)
+    (at 208.8134 128.2192 270)
     (descr "Resistance verticale")
     (tags R)
@@
   )
   (module R1 (layer F.Cu)
-    (at 211.3407 128.2319 270)
+    (at 211.836 128.2319 270)
     (descr "Resistance verticale")
     (tags R)
@@
   )
   (module R1 (layer F.Cu)
-    (at 215.6587 129.5019)
+    (at 218.5924 128.2319 270)
     (descr "Resistance verticale")
     (tags R)
     (autoplace_cost90 10)
     (autoplace_cost180 10)
-    (fp_text reference R3 (at 3.9116 0) (layer F.SilkS)
-      (effects (font (size 1.397 1.27) (thickness 0.2032)))
-    )
-    (fp_text value 1M (at 6.5786 -0.1143) (layer F.SilkS) hide
+    (fp_text reference R3 (at 3.9116 0 270) (layer F.SilkS)
+      (effects (font (size 1.397 1.27) (thickness 0.2032)))
+    )
+    (fp_text value 1M (at 6.5786 -0.1143 270) (layer F.SilkS) hide
       (effects (font (size 1.397 1.27) (thickness 0.2032)))
     )
     (fp_line (start -1.27 0) (end 1.27 0) (layer F.SilkS) (width 0.381))
     (fp_circle (center -1.27 0) (end -0.635 1.27) (layer F.SilkS) (width 0.381))
-    (pad 1 thru_hole circle (at -1.27 0) (size 1.397 1.397) (drill 0.8128)
+    (pad 1 thru_hole circle (at -1.27 0 270) (size 1.397 1.397) (drill 0.8128)
       (layers *.Cu *.Mask F.SilkS)
       (net 25 /SHIELD)
     )
-    (pad 2 thru_hole circle (at 1.27 0) (size 1.397 1.397) (drill 0.8128)
+    (pad 2 thru_hole circle (at 1.27 0 270) (size 1.397 1.397) (drill 0.8128)
       (layers *.Cu *.Mask F.SilkS)
       (net 27 GND)
@@
     (descr "Connecteurs 2 pins")
     (tags "CONN DEV")
-    (fp_text reference JP1 (at 0 -1.905 270) (layer F.SilkS)
+    (fp_text reference JP1 (at -3.2893 0.0127 360) (layer F.SilkS)
       (effects (font (size 0.762 0.762) (thickness 0.1524)))
     )
-    (fp_text value JUMPER (at 0 -1.905 270) (layer F.SilkS) hide
+    (fp_text value JUMPER (at 3.3528 0.0254 360) (layer F.SilkS) hide
       (effects (font (size 0.762 0.762) (thickness 0.1524)))
     )
@@
     )
   )
+  (gr_line (start 211.836 130.4925) (end 211.8614 130.4925) (angle 90) (layer Dwgs.User) (width 0.2))
+  (gr_line (start 211.836 123.063) (end 211.836 130.4925) (angle 90) (layer Dwgs.User) (width 0.2))
+  (gr_line (start 208.8134 129.8194) (end 208.8642 129.8194) (angle 90) (layer Dwgs.User) (width 0.2))
+  (gr_line (start 208.8134 123.063) (end 208.8134 129.8194) (angle 90) (layer Dwgs.User) (width 0.2))
   (dimension 47.5107 (width 0.3) (layer Dwgs.User)
     (gr_text "47,511 mm" (at 210.34375 162.487599) (layer Dwgs.User)
@@
   (segment (start 204.7494 133.7183) (end 192.6463 133.7183) (width 0.381) (layer B.Cu) (net 2))
   (segment (start 204.7494 133.7183) (end 199.0217 133.7183) (width 0.381) (layer B.Cu) (net 2))
-  (segment (start 209.3214 126.9619) (end 209.3214 123.0757) (width 0.381) (layer B.Cu) (net 3))
+  (segment (start 209.3087 123.063) (end 209.3087 126.4539) (width 0.381) (layer B.Cu) (net 3))
+  (segment (start 209.3087 126.4539) (end 208.8134 126.9492) (width 0.381) (layer B.Cu) (net 3))
   (segment (start 209.3214 123.0757) (end 209.3087 123.063) (width 0.381) (layer B.Cu) (net 3))
-  (segment (start 211.3407 126.9619) (end 211.3407 123.063) (width 0.381) (layer B.Cu) (net 4))
+  (segment (start 211.3407 123.063) (end 211.3407 126.4666) (width 0.381) (layer B.Cu) (net 4))
+  (segment (start 211.3407 126.4666) (end 211.836 126.9619) (width 0.381) (layer B.Cu) (net 4))
   (segment (start 217.6399 140.5636) (end 217.6399 141.7193) (width 0.381) (layer B.Cu) (net 5))
   (segment (start 221.9706 143.5735) (end 224.2185 145.8214) (width 0.381) (layer B.Cu) (net 5))
@@
   (segment (start 203.1238 142.963898) (end 208.545018 142.963898) (width 0.381) (layer B.Cu) (net 12))
   (segment (start 207.2894 134.9883) (end 201.8538 134.9883) (width 0.381) (layer F.Cu) (net 13))
-  (segment (start 201.8284 134.9883) (end 198.628 134.9883) (width 0.381) (layer B.Cu) (net 13) (status 800000))
+  (segment (start 201.8284 134.9883) (end 198.628 134.9883) (width 0.381) (layer B.Cu) (net 13))
   (segment (start 201.8411 134.9756) (end 201.8284 134.9883) (width 0.381) (layer B.Cu) (net 13))
   (via (at 201.8411 134.9756) (size 1.524) (layers F.Cu B.Cu) (net 13))
@@
   (segment (start 206.72552 131.7117) (end 204.5589 131.7117) (width 0.381) (layer B.Cu) (net 24))
   (segment (start 199.3646 131.7117) (end 198.628 132.4483) (width 0.381) (layer B.Cu) (net 24))
-  (segment (start 214.3887 126.9619) (end 214.3887 129.5019) (width 0.508) (layer B.Cu) (net 25))
-  (segment (start 217.4367 120.396) (end 217.4367 123.9139) (width 0.508) (layer B.Cu) (net 25))
-  (segment (start 217.4367 123.9139) (end 214.3887 126.9619) (width 0.508) (layer B.Cu) (net 25))
+  (segment (start 218.5924 126.9619) (end 215.3412 126.9619) (width 0.508) (layer B.Cu) (net 25))
+  (segment (start 218.5924 126.9619) (end 218.5924 121.5517) (width 0.508) (layer B.Cu) (net 25))
+  (segment (start 218.5924 121.5517) (end 217.4367 120.396) (width 0.508) (layer B.Cu) (net 25))
   (segment (start 203.7207 120.396) (end 217.4367 120.396) (width 0.508) (layer B.Cu) (net 25))
   (segment (start 228.1809 145.8087) (end 228.1809 144.9451) (width 0.381) (layer B.Cu) (net 26))
@@
   (segment (start 218.3003 139.1285) (end 216.08542 136.91362) (width 0.381) (layer B.Cu) (net 26))
   (segment (start 218.3003 141.122398) (end 218.3003 139.1285) (width 0.381) (layer B.Cu) (net 26))
+  (segment (start 206.7687 123.063) (end 206.7687 124.2949) (width 0.508) (layer B.Cu) (net 27))
+  (segment (start 206.7687 124.2949) (end 204.1017 126.9619) (width 0.508) (layer B.Cu) (net 27))
+  (segment (start 206.7687 123.063) (end 206.6544 123.063) (width 0.508) (layer B.Cu) (net 27))
   (segment (start 210.74888 135.31342) (end 205.7146 140.3477) (width 0.508) (layer B.Cu) (net 27))
   (segment (start 214.31504 135.31342) (end 210.74888 135.31342) (width 0.508) (layer B.Cu) (net 27))
@@
   (segment (start 220.3958 133.71322) (end 220.8276 133.71322) (width 0.381) (layer B.Cu) (net 28))
   (segment (start 220.8276 133.71322) (end 221.93758 133.71322) (width 0.381) (layer B.Cu) (net 28))
-  (segment (start 210.72348 131.7117) (end 210.72348 130.11912) (width 0.381) (layer B.Cu) (net 29))
-  (segment (start 210.72348 130.11912) (end 211.3407 129.5019) (width 0.381) (layer B.Cu) (net 29))
-  (segment (start 209.92592 131.7117) (end 209.92592 130.10642) (width 0.381) (layer B.Cu) (net 30))
-  (segment (start 209.92592 130.10642) (end 209.3214 129.5019) (width 0.381) (layer B.Cu) (net 30))
-  (segment (start 208.32572 131.7117) (end 208.32572 130.32232) (width 0.381) (layer B.Cu) (net 31))
-  (segment (start 207.5053 129.5019) (end 206.7687 129.5019) (width 0.381) (layer B.Cu) (net 31))
-  (segment (start 208.32572 130.32232) (end 207.5053 129.5019) (width 0.381) (layer B.Cu) (net 31))
+  (segment (start 210.72348 131.7117) (end 210.72348 130.61442) (width 0.381) (layer B.Cu) (net 29))
+  (segment (start 210.72348 130.61442) (end 211.836 129.5019) (width 0.381) (layer B.Cu) (net 29))
+  (segment (start 209.92592 131.7117) (end 209.92592 130.60172) (width 0.381) (layer B.Cu) (net 30))
+  (segment (start 209.92592 130.60172) (end 208.8134 129.4892) (width 0.381) (layer B.Cu) (net 30))
+  (segment (start 204.1017 129.5019) (end 207.1751 129.5019) (width 0.381) (layer B.Cu) (net 31))
+  (segment (start 208.32572 130.65252) (end 208.32572 131.7117) (width 0.381) (layer B.Cu) (net 31))
+  (segment (start 207.1751 129.5019) (end 208.32572 130.65252) (width 0.381) (layer B.Cu) (net 31))
   (segment (start 225.9584 136.652) (end 230.3526 136.652) (width 0.381) (layer B.Cu) (net 32))
   (segment (start 221.6404 134.51332) (end 223.81972 134.51332) (width 0.381) (layer B.Cu) (net 32))
